File: hw/power.sch (KiCad schematic (older format))
At the start: 9 parts, among them Q1 Q_PMOS_GSD, U1 ME2188AXXPG

Commit message: epd-clock: hw v0.2
Parts:
- removed R1, R3: 0, Resistor_SMD:R_0603_1608Metric, symbol Device:R
- added JP1, JP2: Jumper, Jumper:SolderJumper-2_P1.3mm_Open_RoundedPad1.0x1.5mm, symbol Device:Jumper
- C2: footprint Capacitor_SMD:C_0805_2012Metric -> Capacitor_SMD:C_1206_3216Metric
- renumbered R2 to R1
Connections:
- net +3V3: now also JP2.2
- net at C2.1, U1.2 (Vout): now also JP2.1
- net at C1.1, L1.1, Q1.2 (S): now also JP1.2
- net at BT1.1 (+): now also JP1.1
Other:
- moved on the sheet: BT1
Changed lines of the file:
@@
 	5000 4150 5000 3900
-$Comp
-L Device:C C?
-U 1 1 60F0A28F
-P 6500 3750
-AR Path="/60F0A28F" Ref="C?"  Part="1"
-AR Path="/60F00547/60F0A28F" Ref="C2"  Part="1"
-F 0 "C2" H 6615 3796 50  0000 L CNN
-F 1 "100uF" H 6615 3705 50  0000 L CNN
-F 2 "Capacitor_SMD:C_0805_2012Metric" H 6538 3600 50  0001 C CNN
-F 3 "~" H 6500 3750 50  0001 C CNN
-	1    6500 3750
-	1    0    0    -1
-$EndComp
 $Comp
 L Device:L L?
@@
 	4550 3000 4550 3500
 $Comp
-L Device:R R2
+L Device:R R1
 U 1 1 60FDE5DB
 P 5950 3000
-F 0 "R2" V 5743 3000 50  0000 C CNN
+F 0 "R1" V 5743 3000 50  0000 C CNN
 F 1 "10K" V 5834 3000 50  0000 C CNN
 F 2 "Resistor_SMD:R_0603_1608Metric" V 5880 3000 50  0001 C CNN
@@
 ADEN#
 $Comp
-L power:GND #PWR03
+L power:GND #PWR02
 U 1 1 6113514D
 P 6800 4150
-F 0 "#PWR03" H 6800 3900 50  0001 C CNN
+F 0 "#PWR02" H 6800 3900 50  0001 C CNN
 F 1 "GND" V 6805 4022 50  0000 R CNN
 F 2 "" H 6800 4150 50  0001 C CNN
@@
 $EndComp
 $Comp
-L power:+3V3 #PWR02
+L power:+3V3 #PWR03
 U 1 1 6113576C
-P 6800 3500
-F 0 "#PWR02" H 6800 3350 50  0001 C CNN
-F 1 "+3V3" V 6815 3628 50  0000 L CNN
-F 2 "" H 6800 3500 50  0001 C CNN
-F 3 "" H 6800 3500 50  0001 C CNN
-	1    6800 3500
+P 7250 3500
+F 0 "#PWR03" H 7250 3350 50  0001 C CNN
+F 1 "+3V3" V 7265 3628 50  0000 L CNN
+F 2 "" H 7250 3500 50  0001 C CNN
+F 3 "" H 7250 3500 50  0001 C CNN
+	1    7250 3500
 	0    1    1    0
 $EndComp
@@
 L Device:Battery_Cell BT1
 U 1 1 61256DF8
-P 4200 3850
-F 0 "BT1" H 4318 3946 50  0000 L CNN
-F 1 "Battery_Cell" H 4318 3855 50  0000 L CNN
-F 2 "custom:AAA_holder_smt" V 4200 3910 50  0001 C CNN
-F 3 "~" V 4200 3910 50  0001 C CNN
-	1    4200 3850
+P 3900 3850
+F 0 "BT1" H 4018 3946 50  0000 L CNN
+F 1 "Battery_Cell" H 4018 3855 50  0000 L CNN
+F 2 "custom:AAA_holder_smt" V 3900 3910 50  0001 C CNN
+F 3 "~" V 3900 3910 50  0001 C CNN
+	1    3900 3850
 	1    0    0    -1
 $EndComp
-Wire Wire Line
-	4200 3500 4200 3650
-Wire Wire Line
-	4200 3950 4200 4150
-Wire Wire Line
-	4200 4150 5000 4150
 $Comp
 L power:PWR_FLAG #FLG01
@@
 	-1   0    0    1
 $EndComp
-$Comp
-L Device:R R1
-U 1 1 610A5E35
-P 4350 3500
-F 0 "R1" V 4250 3500 50  0000 C CNN
-F 1 "0" V 4450 3500 50  0000 C CNN
-F 2 "Resistor_SMD:R_0603_1608Metric" V 4280 3500 50  0001 C CNN
-F 3 "~" H 4350 3500 50  0001 C CNN
-	1    4350 3500
-	0    1    1    0
-$EndComp
 Connection ~ 5000 3500
 Wire Wire Line
@@
 Connection ~ 4550 3500
 $Comp
-L Device:R R3
-U 1 1 610C7213
-P 6650 3500
-F 0 "R3" V 6550 3500 50  0000 C CNN
-F 1 "0" V 6750 3500 50  0000 C CNN
-F 2 "Resistor_SMD:R_0603_1608Metric" V 6580 3500 50  0001 C CNN
-F 3 "~" H 6650 3500 50  0001 C CNN
-	1    6650 3500
-	0    1    1    0
+L power:PWR_FLAG #FLG03
+U 1 1 6117B3D0
+P 7200 3600
+F 0 "#FLG03" H 7200 3675 50  0001 C CNN
+F 1 "PWR_FLAG" H 7200 3773 50  0000 C CNN
+F 2 "" H 7200 3600 50  0001 C CNN
+F 3 "~" H 7200 3600 50  0001 C CNN
+	1    7200 3600
+	-1   0    0    1
 $EndComp
+$Comp
+L Device:Jumper JP2
+U 1 1 6117C3CD
+P 6850 3500
+F 0 "JP2" H 6850 3450 50  0000 C CNN
+F 1 "Jumper" H 6850 3400 50  0000 C CNN
+F 2 "Jumper:SolderJumper-2_P1.3mm_Open_RoundedPad1.0x1.5mm" H 6850 3500 50  0001 C CNN
+F 3 "~" H 6850 3500 50  0001 C CNN
+	1    6850 3500
+	1    0    0    -1
+$EndComp
+Wire Wire Line
+	7150 3500 7200 3500
+Wire Wire Line
+	7200 3600 7200 3500
+Connection ~ 7200 3500
+Wire Wire Line
+	7200 3500 7250 3500
+Wire Wire Line
+	6550 3500 6500 3500
 Connection ~ 6500 3500
+$Comp
+L Device:Jumper JP1
+U 1 1 611863AB
+P 4200 3500
+F 0 "JP1" H 4200 3450 50  0000 C CNN
+F 1 "Jumper" H 4200 3400 50  0000 C CNN
+F 2 "Jumper:SolderJumper-2_P1.3mm_Open_RoundedPad1.0x1.5mm" H 4200 3500 50  0001 C CNN
+F 3 "~" H 4200 3500 50  0001 C CNN
+	1    4200 3500
+	1    0    0    -1
+$EndComp
+Wire Wire Line
+	3900 3650 3900 3500
+Wire Wire Line
+	3900 3950 3900 4150
+Wire Wire Line
+	3900 4150 5000 4150
+$Comp
+L Device:C C2
+U 1 1 611EE99D
+P 6500 3750
+F 0 "C2" H 6615 3796 50  0000 L CNN
+F 1 "100uF" H 6615 3705 50  0000 L CNN
+F 2 "Capacitor_SMD:C_1206_3216Metric" H 6538 3600 50  0001 C CNN
+F 3 "~" H 6500 3750 50  0001 C CNN
+	1    6500 3750
+	1    0    0    -1
+$EndComp
 $EndSCHEMATC
