File: hw/button.sch (KiCad schematic (older format))
At the start: 6 parts, among them SW1 SW_Push, SW2 SW_Push, SW3 SW_Push

Commit message: epd-clock: hw v0.2
Parts:
- renumbered R11 to R10, R12 to R11, R13 to R12
Changed lines of the file:
@@
 $EndComp
 $Comp
-L Device:R R11
+L Device:R R10
 U 1 1 61233949
 P 5350 2800
-F 0 "R11" V 5143 2800 50  0000 C CNN
+F 0 "R10" V 5143 2800 50  0000 C CNN
 F 1 "10K" V 5234 2800 50  0000 C CNN
 F 2 "Resistor_SMD:R_0603_1608Metric" V 5280 2800 50  0001 C CNN
@@
 $EndComp
 $Comp
-L Device:R R12
+L Device:R R11
 U 1 1 6123418A
 P 5350 3250
-F 0 "R12" V 5143 3250 50  0000 C CNN
+F 0 "R11" V 5143 3250 50  0000 C CNN
 F 1 "10K" V 5234 3250 50  0000 C CNN
 F 2 "Resistor_SMD:R_0603_1608Metric" V 5280 3250 50  0001 C CNN
@@
 $EndComp
 $Comp
-L Device:R R13
+L Device:R R12
 U 1 1 612344CD
 P 5350 3700
-F 0 "R13" V 5143 3700 50  0000 C CNN
+F 0 "R12" V 5143 3700 50  0000 C CNN
 F 1 "10K" V 5234 3700 50  0000 C CNN
 F 2 "Resistor_SMD:R_0603_1608Metric" V 5280 3700 50  0001 C CNN
@@
 BT2
 $Comp
-L power:+3V3 #PWR043
+L power:+3V3 #PWR046
 U 1 1 610A0EA0
 P 5050 2800
-F 0 "#PWR043" H 5050 2650 50  0001 C CNN
+F 0 "#PWR046" H 5050 2650 50  0001 C CNN
 F 1 "+3V3" H 5065 2973 50  0000 C CNN
 F 2 "" H 5050 2800 50  0001 C CNN
@@
 Connection ~ 5050 2800
 $Comp
-L power:GND #PWR044
+L power:GND #PWR047
 U 1 1 610A3FCD
 P 6050 2800
-F 0 "#PWR044" H 6050 2550 50  0001 C CNN
+F 0 "#PWR047" H 6050 2550 50  0001 C CNN
 F 1 "GND" V 6055 2672 50  0000 R CNN
 F 2 "" H 6050 2800 50  0001 C CNN
@@
 $EndComp
 $Comp
-L power:GND #PWR045
+L power:GND #PWR048
 U 1 1 610A4511
 P 6050 3250
-F 0 "#PWR045" H 6050 3000 50  0001 C CNN
+F 0 "#PWR048" H 6050 3000 50  0001 C CNN
 F 1 "GND" V 6055 3122 50  0000 R CNN
 F 2 "" H 6050 3250 50  0001 C CNN
@@
 $EndComp
 $Comp
-L power:GND #PWR046
+L power:GND #PWR049
 U 1 1 610A4989
 P 6050 3700
-F 0 "#PWR046" H 6050 3450 50  0001 C CNN
+F 0 "#PWR049" H 6050 3450 50  0001 C CNN
 F 1 "GND" V 6055 3572 50  0000 R CNN
 F 2 "" H 6050 3700 50  0001 C CNN

Commit message: epd-clock: hw: v0.2
Parts:
- renumbered R10 to R15, R11 to R16, R12 to R17
Changed lines of the file:
@@
 $EndComp
 $Comp
-L Device:R R10
+L Device:R R15
 U 1 1 61233949
 P 5350 2800
-F 0 "R10" V 5143 2800 50  0000 C CNN
+F 0 "R15" V 5143 2800 50  0000 C CNN
 F 1 "10K" V 5234 2800 50  0000 C CNN
 F 2 "Resistor_SMD:R_0603_1608Metric" V 5280 2800 50  0001 C CNN
@@
 $EndComp
 $Comp
-L Device:R R11
+L Device:R R16
 U 1 1 6123418A
 P 5350 3250
-F 0 "R11" V 5143 3250 50  0000 C CNN
+F 0 "R16" V 5143 3250 50  0000 C CNN
 F 1 "10K" V 5234 3250 50  0000 C CNN
 F 2 "Resistor_SMD:R_0603_1608Metric" V 5280 3250 50  0001 C CNN
@@
 $EndComp
 $Comp
-L Device:R R12
+L Device:R R17
 U 1 1 612344CD
 P 5350 3700
-F 0 "R12" V 5143 3700 50  0000 C CNN
+F 0 "R17" V 5143 3700 50  0000 C CNN
 F 1 "10K" V 5234 3700 50  0000 C CNN
 F 2 "Resistor_SMD:R_0603_1608Metric" V 5280 3700 50  0001 C CNN
@@
 BT2
 $Comp
-L power:+3V3 #PWR046
+L power:+3V3 #PWR044
 U 1 1 610A0EA0
 P 5050 2800
-F 0 "#PWR046" H 5050 2650 50  0001 C CNN
+F 0 "#PWR044" H 5050 2650 50  0001 C CNN
 F 1 "+3V3" H 5065 2973 50  0000 C CNN
 F 2 "" H 5050 2800 50  0001 C CNN
@@
 Connection ~ 5050 2800
 $Comp
-L power:GND #PWR047
+L power:GND #PWR045
 U 1 1 610A3FCD
 P 6050 2800
-F 0 "#PWR047" H 6050 2550 50  0001 C CNN
+F 0 "#PWR045" H 6050 2550 50  0001 C CNN
 F 1 "GND" V 6055 2672 50  0000 R CNN
 F 2 "" H 6050 2800 50  0001 C CNN
@@
 $EndComp
 $Comp
-L power:GND #PWR048
+L power:GND #PWR046
 U 1 1 610A4511
 P 6050 3250
-F 0 "#PWR048" H 6050 3000 50  0001 C CNN
+F 0 "#PWR046" H 6050 3000 50  0001 C CNN
 F 1 "GND" V 6055 3122 50  0000 R CNN
 F 2 "" H 6050 3250 50  0001 C CNN
@@
 $EndComp
 $Comp
-L power:GND #PWR049
+L power:GND #PWR047
 U 1 1 610A4989
 P 6050 3700
-F 0 "#PWR049" H 6050 3450 50  0001 C CNN
+F 0 "#PWR047" H 6050 3450 50  0001 C CNN
 F 1 "GND" V 6055 3572 50  0000 R CNN
 F 2 "" H 6050 3700 50  0001 C CNN

Commit message: hw: 合并电源网络
取消墨水屏电源控制mos与独立电源域，墨水屏使用深度休眠模式，共用主
电源域。
Parts:
- renumbered R15 to R12, R16 to R13, R17 to R14
Changed lines of the file:
@@
 $EndComp
 $Comp
-L Device:R R15
+L Device:R R12
 U 1 1 61233949
 P 5350 2800
-F 0 "R15" V 5143 2800 50  0000 C CNN
+F 0 "R12" V 5143 2800 50  0000 C CNN
 F 1 "10K" V 5234 2800 50  0000 C CNN
 F 2 "Resistor_SMD:R_0603_1608Metric" V 5280 2800 50  0001 C CNN
@@
 $EndComp
 $Comp
-L Device:R R16
+L Device:R R13
 U 1 1 6123418A
 P 5350 3250
-F 0 "R16" V 5143 3250 50  0000 C CNN
+F 0 "R13" V 5143 3250 50  0000 C CNN
 F 1 "10K" V 5234 3250 50  0000 C CNN
 F 2 "Resistor_SMD:R_0603_1608Metric" V 5280 3250 50  0001 C CNN
@@
 $EndComp
 $Comp
-L Device:R R17
+L Device:R R14
 U 1 1 612344CD
 P 5350 3700
-F 0 "R17" V 5143 3700 50  0000 C CNN
+F 0 "R14" V 5143 3700 50  0000 C CNN
 F 1 "10K" V 5234 3700 50  0000 C CNN
 F 2 "Resistor_SMD:R_0603_1608Metric" V 5280 3700 50  0001 C CNN
@@
 BT2
 $Comp
-L power:+3V3 #PWR044
+L power:+3V3 #PWR042
 U 1 1 610A0EA0
 P 5050 2800
-F 0 "#PWR044" H 5050 2650 50  0001 C CNN
+F 0 "#PWR042" H 5050 2650 50  0001 C CNN
 F 1 "+3V3" H 5065 2973 50  0000 C CNN
 F 2 "" H 5050 2800 50  0001 C CNN
@@
 Connection ~ 5050 2800
 $Comp
-L power:GND #PWR045
+L power:GND #PWR043
 U 1 1 610A3FCD
 P 6050 2800
-F 0 "#PWR045" H 6050 2550 50  0001 C CNN
+F 0 "#PWR043" H 6050 2550 50  0001 C CNN
 F 1 "GND" V 6055 2672 50  0000 R CNN
 F 2 "" H 6050 2800 50  0001 C CNN
@@
 $EndComp
 $Comp
-L power:GND #PWR046
+L power:GND #PWR044
 U 1 1 610A4511
 P 6050 3250
-F 0 "#PWR046" H 6050 3000 50  0001 C CNN
+F 0 "#PWR044" H 6050 3000 50  0001 C CNN
 F 1 "GND" V 6055 3122 50  0000 R CNN
 F 2 "" H 6050 3250 50  0001 C CNN
@@
 $EndComp
 $Comp
-L power:GND #PWR047
+L power:GND #PWR045
 U 1 1 610A4989
 P 6050 3700
-F 0 "#PWR047" H 6050 3450 50  0001 C CNN
+F 0 "#PWR045" H 6050 3450 50  0001 C CNN
 F 1 "GND" V 6055 3572 50  0000 R CNN
 F 2 "" H 6050 3700 50  0001 C CNN
